Commit message: ros2 control

File: rb1_description/robot/rb1_simple.urdf (robot description, URDF)
Before this commit: robot my_rb1_robot, 10 links, 9 joints
Links:
- added link elevator_link, mass 100; collision cylinder length=0.005 radius=0.25; visual cylinder length=0.005 radius=0.25
- link arrow_link: geometry visual box size=0.4 0.1 0.001
- link arrow_link_2: geometry visual box size=0.15 0.1 0.001
- link arrow_link_3: geometry visual box size=0.15 0.1 0.001
Joints:
- removed joint base_to_arrow
- added joint elevator_joint: type prismatic, parent base_link, child elevator_link, origin xyz=0 0 0.16 rpy=0 0 0, axis 0 0 1, limit lower=0 upper=2 effort=10000 velocity=0.1
- added joint elevator_to_arrow: type fixed, parent elevator_link, child arrow_link, origin xyz=0.0 0.0 0.0025
