Commit message: modified physics to pick up cart

File: rb1_ros2_description/urdf/elevator/elevator.urdf.xacro (robot description, xacro)
@@ -27,7 +27,7 @@
 		</inertial-->
 		<inertial>
-			<mass value="0.005" />
+			<mass value="2" />
 			<origin xyz="0 0 -0.27" />
-			<xacro:solid_cuboid_inertia1 m="0.005" h="0.05" d="0.05" w="0.05"/>
+			<xacro:solid_cuboid_inertia1 m="2" h="0.05" d="0.05" w="0.05"/>
 		</inertial>
 		<visual>
@@ -60,6 +60,6 @@
 			<child link="${prefix}_platform_link" />
 			<axis xyz="0 0 1"/>
-			<limit effort="100.0" lower="0.0" upper="0.034" velocity="0.5"/>
-            <dynamics damping="0.1" friction="1.0"/>
+			<limit effort="1000.0" lower="0.0" upper="0.034" velocity="0.05"/>
+            <dynamics damping="0.9" friction="1.0"/>
             <!-- upper="0.034 -->
 	</joint>
@@ -71,8 +71,8 @@
 		</inertial-->
 		<inertial>
-			<mass value="0.005" />
+			<mass value="2" />
 			<origin xyz="0 0 -0.27" />
 			<!-- <solid_cuboid_inertia m="0.005" h="0.05" d="0.05" w="0.05"/> -->
-            <xacro:solid_cuboid_inertia1 m="0.005" h="0.05" d="0.05" w="0.05"/>
+            <xacro:solid_cuboid_inertia1 m="2" h="0.05" d="0.05" w="0.05"/>
 		</inertial>
 		<visual>
@@ -94,4 +94,5 @@
 		<collision>
 			<origin xyz="0 0 0" rpy="0 0 0 " />
+			<mass>2</mass>
 			<geometry>
 				<mesh filename="package://rb1_ros2_description/meshes/elevator/rb1_elevator_platform.dae"/>
